Commit message: week2 assignment2

File: src/hrwros_week2/urdf/hrwros_assignment2.xacro (robot description, xacro)
@@ -71,4 +71,11 @@
     <origin xyz="0 0 0.6" rpy="0 0 ${radians(90)}" />
   </joint>
-  <!-- Add your solution to assignment 2 here -->
+  <!-- sphere -->
+  <xacro:include filename="$(find hrwros_week2)/urdf/sphere/sphere.urdf.xacro" />
+  <xacro:sphere_urdf prefix="sphere_1_" radi="0.4" />
+  <joint name="sphere1_joint" type="fixed">
+    <parent link="world" />
+    <child link="sphere_1_base_link" />
+    <origin xyz="5.5 -4.5 0.4" />
+  </joint>
 </robot>
