Commit message: Week3 Assignment3

File: src/hrwros_support/urdf/robot_system/robot_system.gazebo.xacro (robot description, xacro)
@@ -23,4 +23,7 @@
       <turnGravityOff>true</turnGravityOff>
     </gazebo>
+    <gazebo reference="${robot_prefix}ee_link">
+      <turnGravityOff>true</turnGravityOff>
+    </gazebo>
     <gazebo>
       <plugin name="gazebo_ros_control" filename="libgazebo_ros_control.so">

File: src/hrwros_support/urdf/vacuum_gripper/vacuum_gripper.urdf.xacro (robot description, xacro)
@@ -22,8 +22,8 @@
       <inertial>
         <origin xyz="0 0 0" rpy="0 0 0" />
-        <inertia ixx="1.0" ixy="0" ixz="0"
-                 iyy="1.0" iyz="0"
-                 izz="1.0" />
-        <mass value="1.0" />
+        <inertia ixx="0.00001" ixy="0" ixz="0"
+                 iyy="0.00001" iyz="0"
+                 izz="0.00001" />
+        <mass value="0.00001" />
       </inertial>
     </link>
